File: board/hakkaa.kicad_pcb (KiCad board)
At the start: 2 copper layers, 78 x 83.7 mm, 22 parts, among them SW1 SW_Push, U1 ESP32-C3_SUPERMINI_SMD, U2 ShakeSensor

Commit message: Prepare for publication
Other:
- board text added: "hakkā board"
- board text added: "https://github.com/hakkaatachi"
- board text added: "©2025 Ulf Wetzker CERN-OHL-W v2.0 https://cern-ohl.web.cern.ch/"
